File: esp32_lan8720_spacer.kicad/lan8720_spacer.kicad_pcb (KiCad board)
At the start: 2 copper layers, 20.1 x 25.8 mm, 3 parts, among them J1 Conn_02x07_Odd_Even, J2 Conn_02x07_Odd_Even

Commit message: kicad files for v1.1 PCB
Parts:
- G***: moved to F.Cu
- J1: moved to B.Cu
- J2: footprint Connector_PinSocket_2.54mm:PinSocket_2x07_P2.54mm_Vertical -> ct:PinSocket_2x07_P2.54_Vertical_Hybrid_SMD_THT; moved to B.Cu
- moved G*** 64.1 mm to (245.9, 70.5), turned to 0 degrees
- moved J2 49.9 mm to (239.0, 71.4), turned to 0 degrees
- moved J1 41.4 mm to (231.4, 89.9)
Connections:
- J1 pad 1: /3v3 -> /TX1
- J1 pad 10: /RX0 -> /MDC
- J1 pad 11: /TX0 -> /GND
- J1 pad 12: /TXEN -> /GND
- J1 pad 13: /NC -> /3v3
- J1 pad 14: /TX1 -> /3v3
- J1 pad 2: /3v3 -> /NC
- J1 pad 3: /GND -> /TXEN
- J1 pad 4: /GND -> /TX0
- J1 pad 5: /MDC -> /RX0
- J1 pad 6: /MDIO -> /RX1
- J1 pad 7: /CRS -> /RETCLK
- J1 pad 8: /RETCLK -> /CRS
- J1 pad 9: /RX1 -> /MDIO
- J2 pad 1: /3v3 -> /NC
- J2 pad 10: /RX0 -> /MDIO
- J2 pad 11: /TX0 -> /GND
- J2 pad 12: /TXEN -> /GND
- J2 pad 13: /NC -> /3v3
- J2 pad 14: /TX1 -> /3v3
- J2 pad 2: /3v3 -> /TX1
- J2 pad 3: /GND -> /TX0
- J2 pad 4: /GND -> /TXEN
- J2 pad 5: /MDC -> /RX1
- J2 pad 6: /MDIO -> /RX0
- J2 pad 9: /RX1 -> /MDC
Routing:
- net /GND: track 18.1 -> 44.4 mm
- net /3v3: track 15.1 -> 36.1 mm
- net /NC: track 10.0 -> 24.3 mm, vias 0 -> 1
- net /TX0: track 11.4 -> 25.3 mm
- net /RX1: track 15.4 -> 28.4 mm
- net /MDC: track 16.7 -> 27.1 mm
- net /TXEN: track 17.1 -> 27.1 mm
- net /CRS: track 41.0 -> 31.6 mm
- net /RETCLK: track 36.7 -> 30.2 mm
- net /RX0: track 29.9 -> 33.9 mm
- net /MDIO: track 29.7 -> 32.0 mm
- net /TX1: track 15.5 -> 17.3 mm
Other:
- board size 20.1 x 25.8 mm -> 25 x 26.7 mm
- board text added: "${TITLE} ${REVISION}"
