File: esp32_lan8720_spacer.kicad/lan8720_spacer.kicad_sch (KiCad schematic)
At the start: 2 parts, among them J1 Conn_02x07_Odd_Even, J2 Conn_02x07_Odd_Even

Commit message: kicad files for v1.1 PCB
Parts:
- J2: footprint Connector_PinSocket_2.54mm:PinSocket_2x07_P2.54mm_Vertical -> ct:PinSocket_2x07_P2.54_Vertical_Hybrid_SMD_THT
Connections:
- net 3v3: now also J1.13 (Pin_13), J1.14 (Pin_14), J2.13 (Pin_13), J2.14 (Pin_14); no longer J1.1 (Pin_1), J1.2 (Pin_2), J2.1 (Pin_1), J2.2 (Pin_2)
- net CRS: now also J1.8 (Pin_8); no longer J1.7 (Pin_7)
- net GND: now also J1.11 (Pin_11), J1.12 (Pin_12), J2.11 (Pin_11), J2.12 (Pin_12); no longer J1.3 (Pin_3), J1.4 (Pin_4), J2.3 (Pin_3), J2.4 (Pin_4)
- net MDC: now also J1.10 (Pin_10), J2.9 (Pin_9); no longer J1.5 (Pin_5), J2.5 (Pin_5)
- net MDIO: now also J1.9 (Pin_9), J2.10 (Pin_10); no longer J1.6 (Pin_6), J2.6 (Pin_6)
- net NC: now also J1.2 (Pin_2), J2.1 (Pin_1); no longer J1.13 (Pin_13), J2.13 (Pin_13)
- net RETCLK: now also J1.7 (Pin_7); no longer J1.8 (Pin_8)
- net RX0: now also J1.5 (Pin_5), J2.6 (Pin_6); no longer J1.10 (Pin_10), J2.10 (Pin_10)
- net RX1: now also J1.6 (Pin_6), J2.5 (Pin_5); no longer J1.9 (Pin_9), J2.9 (Pin_9)
- net TX0: now also J1.4 (Pin_4), J2.3 (Pin_3); no longer J1.11 (Pin_11), J2.11 (Pin_11)
- net TX1: now also J1.1 (Pin_1), J2.2 (Pin_2); no longer J1.14 (Pin_14), J2.14 (Pin_14)
- net TXEN: now also J1.3 (Pin_3), J2.4 (Pin_4); no longer J1.12 (Pin_12), J2.12 (Pin_12)
Other:
- moved on the sheet: J2
Changed lines of the file:
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@@
   (title_block
     (title "ESP32 LAN8720 Spacer")
-    (date "24/09/2022")
-    (rev "v1.0")
+    (date "2022-10-17")
+    (rev "v1.1")
     (company "ColossalTurtle")
   )
@@
     (stroke (width 0) (type default) (color 0 0 0 0))
   )
-  (wire (pts (xy 134.62 91.44) (xy 139.7 91.44))
-    (stroke (width 0) (type default) (color 0 0 0 0))
-  )
-  (wire (pts (xy 152.4 96.52) (xy 156.21 96.52))
+  (wire (pts (xy 133.985 86.995) (xy 139.065 86.995))
+    (stroke (width 0) (type default) (color 0 0 0 0))
+  )
+  (wire (pts (xy 151.765 92.075) (xy 155.575 92.075))
     (stroke (width 0) (type default) (color 0 0 0 0))
   )
@@
     (stroke (width 0) (type default) (color 0 0 0 0))
   )
-  (wire (pts (xy 134.62 93.98) (xy 139.7 93.98))
+  (wire (pts (xy 133.985 89.535) (xy 139.065 89.535))
     (stroke (width 0) (type default) (color 0 0 0 0))
   )
@@
     (stroke (width 0) (type default) (color 0 0 0 0))
   )
-  (wire (pts (xy 134.62 96.52) (xy 139.7 96.52))
-    (stroke (width 0) (type default) (color 0 0 0 0))
-  )
-  (wire (pts (xy 152.4 93.98) (xy 156.21 93.98))
-    (stroke (width 0) (type default) (color 0 0 0 0))
-  )
-  (wire (pts (xy 152.4 91.44) (xy 156.21 91.44))
-    (stroke (width 0) (type default) (color 0 0 0 0))
-  )
-  (wire (pts (xy 134.62 86.36) (xy 139.7 86.36))
-    (stroke (width 0) (type default) (color 0 0 0 0))
-  )
-  (wire (pts (xy 152.4 99.06) (xy 156.21 99.06))
+  (wire (pts (xy 133.985 92.075) (xy 139.065 92.075))
+    (stroke (width 0) (type default) (color 0 0 0 0))
+  )
+  (wire (pts (xy 151.765 89.535) (xy 155.575 89.535))
+    (stroke (width 0) (type default) (color 0 0 0 0))
+  )
+  (wire (pts (xy 151.765 86.995) (xy 155.575 86.995))
+    (stroke (width 0) (type default) (color 0 0 0 0))
+  )
+  (wire (pts (xy 133.985 81.915) (xy 139.065 81.915))
+    (stroke (width 0) (type default) (color 0 0 0 0))
+  )
+  (wire (pts (xy 151.765 94.615) (xy 155.575 94.615))
     (stroke (width 0) (type default) (color 0 0 0 0))
   )
@@
     (stroke (width 0) (type default) (color 0 0 0 0))
   )
-  (wire (pts (xy 134.62 99.06) (xy 139.7 99.06))
+  (wire (pts (xy 133.985 94.615) (xy 139.065 94.615))
     (stroke (width 0) (type default) (color 0 0 0 0))
   )
@@
     (stroke (width 0) (type default) (color 0 0 0 0))
   )
-  (wire (pts (xy 152.4 86.36) (xy 156.21 86.36))
+  (wire (pts (xy 151.765 81.915) (xy 155.575 81.915))
     (stroke (width 0) (type default) (color 0 0 0 0))
   )
@@
     (stroke (width 0) (type default) (color 0 0 0 0))
   )
-  (wire (pts (xy 134.62 101.6) (xy 139.7 101.6))
+  (wire (pts (xy 133.985 97.155) (xy 139.065 97.155))
     (stroke (width 0) (type default) (color 0 0 0 0))
   )
@@
     (stroke (width 0) (type default) (color 0 0 0 0))
   )
-  (wire (pts (xy 134.62 88.9) (xy 139.7 88.9))
-    (stroke (width 0) (type default) (color 0 0 0 0))
-  )
-  (wire (pts (xy 152.4 88.9) (xy 156.21 88.9))
-    (stroke (width 0) (type default) (color 0 0 0 0))
-  )
-  (wire (pts (xy 152.4 101.6) (xy 156.21 101.6))
+  (wire (pts (xy 133.985 84.455) (xy 139.065 84.455))
+    (stroke (width 0) (type default) (color 0 0 0 0))
+  )
+  (wire (pts (xy 151.765 84.455) (xy 155.575 84.455))
+    (stroke (width 0) (type default) (color 0 0 0 0))
+  )
+  (wire (pts (xy 151.765 97.155) (xy 155.575 97.155))
     (stroke (width 0) (type default) (color 0 0 0 0))
   )
@@
     (effects (font (size 1.27 1.27)) (justify right bottom))
   )
-  (label "MDIO" (at 134.62 91.44 180)
+  (label "MDIO" (at 133.985 86.995 180)
     (effects (font (size 1.27 1.27)) (justify right bottom))
   )
@@
     (effects (font (size 1.27 1.27)) (justify left bottom))
   )
-  (label "GND" (at 156.21 88.9 0)
+  (label "GND" (at 155.575 84.455 0)
     (effects (font (size 1.27 1.27)) (justify left bottom))
   )
@@
     (effects (font (size 1.27 1.27)) (justify right bottom))
   )
-  (label "CRS" (at 156.21 93.98 0)
+  (label "CRS" (at 155.575 89.535 0)
     (effects (font (size 1.27 1.27)) (justify left bottom))
   )
@@
     (effects (font (size 1.27 1.27)) (justify left bottom))
   )
-  (label "RETCLK" (at 134.62 93.98 180)
-    (effects (font (size 1.27 1.27)) (justify right bottom))
-  )
-  (label "GND" (at 134.62 88.9 180)
+  (label "RETCLK" (at 133.985 89.535 180)
+    (effects (font (size 1.27 1.27)) (justify right bottom))
+  )
+  (label "GND" (at 133.985 84.455 180)
     (effects (font (size 1.27 1.27)) (justify right bottom))
   )
@@
     (effects (font (size 1.27 1.27)) (justify right bottom))
   )
-  (label "TXEN" (at 134.62 99.06 180)
+  (label "TXEN" (at 133.985 94.615 180)
     (effects (font (size 1.27 1.27)) (justify right bottom))
   )
@@
     (effects (font (size 1.27 1.27)) (justify left bottom))
   )
-  (label "MDC" (at 156.21 91.44 0)
-    (effects (font (size 1.27 1.27)) (justify left bottom))
-  )
-  (label "3v3" (at 134.62 86.36 180)
-    (effects (font (size 1.27 1.27)) (justify right bottom))
-  )
-  (label "TX1" (at 134.62 101.6 180)
-    (effects (font (size 1.27 1.27)) (justify right bottom))
-  )
-  (label "TX0" (at 156.21 99.06 0)
+  (label "MDC" (at 155.575 86.995 0)
+    (effects (font (size 1.27 1.27)) (justify left bottom))
+  )
+  (label "3v3" (at 133.985 81.915 180)
+    (effects (font (size 1.27 1.27)) (justify right bottom))
+  )
+  (label "TX1" (at 133.985 97.155 180)
+    (effects (font (size 1.27 1.27)) (justify right bottom))
+  )
+  (label "TX0" (at 155.575 94.615 0)
     (effects (font (size 1.27 1.27)) (justify left bottom))
   )
@@
     (effects (font (size 1.27 1.27)) (justify right bottom))
   )
-  (label "RX0" (at 134.62 96.52 180)
-    (effects (font (size 1.27 1.27)) (justify right bottom))
-  )
-  (label "NC" (at 156.21 101.6 0)
-    (effects (font (size 1.27 1.27)) (justify left bottom))
-  )
-  (label "3v3" (at 156.21 86.36 0)
+  (label "RX0" (at 133.985 92.075 180)
+    (effects (font (size 1.27 1.27)) (justify right bottom))
+  )
+  (label "NC" (at 155.575 97.155 0)
+    (effects (font (size 1.27 1.27)) (justify left bottom))
+  )
+  (label "3v3" (at 155.575 81.915 0)
     (effects (font (size 1.27 1.27)) (justify left bottom))
   )
@@
     (effects (font (size 1.27 1.27)) (justify right bottom))
   )
-  (label "RX1" (at 156.21 96.52 0)
+  (label "RX1" (at 155.575 92.075 0)
     (effects (font (size 1.27 1.27)) (justify left bottom))
   )
@@
     (effects (font (size 1.27 1.27)) (justify right bottom))
   )
-  (symbol (lib_id "Connector_Generic:Conn_02x07_Odd_Even") (at 147.32 63.5 0) (mirror y) (unit 1)
+  (symbol (lib_id "Connector_Generic:Conn_02x07_Odd_Even") (at 144.78 63.5 0) (mirror x) (unit 1)
     (in_bom yes) (on_board yes) (fields_autoplaced)
     (property "Reference" "J1" (id 0) (at 146.05 49.53 0))
     (property "Value" "Conn_02x07_Odd_Even" (id 1) (at 146.05 52.07 0))
-    (property "Footprint" "Connector_PinHeader_2.54mm:PinHeader_2x07_P2.54mm_Horizontal" (id 2) (at 147.32 63.5 0)
-      (effects (font (size 1.27 1.27)) hide)
-    )
-    (property "Datasheet" "~" (id 3) (at 147.32 63.5 0)
+    (property "Footprint" "Connector_PinHeader_2.54mm:PinHeader_2x07_P2.54mm_Horizontal" (id 2) (at 144.78 63.5 0)
+      (effects (font (size 1.27 1.27)) hide)
+    )
+    (property "Datasheet" "~" (id 3) (at 144.78 63.5 0)
       (effects (font (size 1.27 1.27)) hide)
     )
@@
     (pin "9")
   )
-  (symbol (lib_id "Connector_Generic:Conn_02x07_Odd_Even") (at 147.32 93.98 0) (mirror y) (unit 1)
+  (symbol (lib_id "Connector_Generic:Conn_02x07_Odd_Even") (at 146.685 89.535 180) (unit 1)
     (in_bom yes) (on_board yes) (fields_autoplaced)
-    (property "Reference" "J2" (id 0) (at 146.05 80.01 0))
-    (property "Value" "Conn_02x07_Odd_Even" (id 1) (at 146.05 82.55 0))
-    (property "Footprint" "Connector_PinSocket_2.54mm:PinSocket_2x07_P2.54mm_Vertical" (id 2) (at 147.32 93.98 0)
-      (effects (font (size 1.27 1.27)) hide)
-    )
-    (property "Datasheet" "~" (id 3) (at 147.32 93.98 0)
+    (property "Reference" "J2" (id 0) (at 145.415 74.93 0))
+    (property "Value" "Conn_02x07_Odd_Even" (id 1) (at 145.415 77.47 0))
+    (property "Footprint" "ct:PinSocket_2x07_P2.54_Vertical_Hybrid_SMD_THT" (id 2) (at 146.685 89.535 0)
+      (effects (font (size 1.27 1.27)) hide)
+    )
+    (property "Datasheet" "~" (id 3) (at 146.685 89.535 0)
       (effects (font (size 1.27 1.27)) hide)
     )
@@
     )
     (path "/7bf4b767-ff56-4cba-af0e-f111782ec127"
-      (reference "J2") (unit 1) (value "Conn_02x07_Odd_Even") (footprint "Connector_PinSocket_2.54mm:PinSocket_2x07_P2.54mm_Vertical")
-    )
-  )
+      (reference "J2") (unit 1) (value "Conn_02x07_Odd_Even") (footprint "ct:PinSocket_2x07_P2.54_Vertical_Hybrid_SMD_THT")
+    )
+  )
