File: esp32_lan8720.kicad/esp32_lan8720.kicad_pcb (KiCad board)
At the start: 2 copper layers, 48 x 84.1 mm, 16 parts, among them J1 Conn_01x19, J2 Conn_02x07_Odd_Even, J3 Conn_01x19, J4 Conn_01x04, J5 Conn_01x04, J6 Screw_Terminal_01x02, J7 Screw_Terminal_01x07

Commit message: kicad files for v1.1 PCB
Parts:
- J2: footprint Connector_PinSocket_2.54mm:PinSocket_2x07_P2.54mm_Vertical -> ct:PinSocket_2x07_P2.54_Vertical_Hybrid_SMD_THT_DBLSIDED
- moved J2 32.5 mm to (135.6, 122.2), turned to 180 degrees
- moved G*** 29.4 mm to (134.6, 105.3)
- moved G*** 29.4 mm to (140.6, 72.0)
- moved J3 29.4 mm to (148.3, 73.0)
- moved J4 29.4 mm to (161.5, 68.5)
- moved J5 29.4 mm to (161.5, 111.7)
- moved J6 29.4 mm to (145.5, 133.7)
- moved J7 29.4 mm to (126.4, 59.3)
- moved TP1 29.4 mm to (152.3, 124.6)
- moved TP4 29.4 mm to (159.2, 117.0)
- moved TP2 29.4 mm to (159.2, 124.8)
- moved J1 29.4 mm to (122.9, 73.0)
- moved JP1 29.4 mm to (122.9, 67.9)
- moved TP3 29.4 mm to (154.1, 117.0)
- moved R1 26.7 mm to (131.6, 116.3)
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Routing:
- net /RETCLK: track 55.0 -> 33.4 mm, vias 2 -> 1
- net /TXEN: track 49.1 -> 53.3 mm
- net /3v3: track 101.1 -> 105.3 mm
- net /GND: track 1.55 -> 5.74 mm
- net /MDIO: track 50.7 -> 54.8 mm
- net /CRS: track 34.5 -> 36.5 mm
- net /RX0: track 53.2 -> 55.2 mm
- net /TX0: track 39.0 -> 40.9 mm
- net /MDC: track 57.6 -> 56.8 mm
- net /RX1: track 39.2 -> 38.7 mm

Commit message: kicad files for v1.2 PCB
Parts:
- added JP2: SolderJumper_2_Open, Jumper:SolderJumper-2_P1.3mm_Open_RoundedPad1.0x1.5mm, F.Cu at (133.3, 119.4)
- added JP3: SolderJumper_2_Open, Jumper:SolderJumper-2_P1.3mm_Open_RoundedPad1.0x1.5mm, F.Cu at (142.2, 119.4)
Connections:
- net /DE renamed /DE/RE
- J3 pad 11: /NC -> /NC_SW
- J3 pad 14: /RETCLK -> /RCLK_SW
Routing:
- net /NC_SW: track 0.00 -> 25.2 mm, vias 0 -> 1
- net /NC: track 30.9 -> 10.3 mm, vias 1 -> 0
- net /RCLK_SW: track 0.00 -> 20.6 mm, vias 0 -> 1
- net /RETCLK: track 33.4 -> 15.7 mm, vias 1 -> 0
