File: esp32_lan8720.kicad/esp32_lan8720.kicad_sch (KiCad schematic)
At the start: 14 parts, among them J1 Conn_01x19, J2 Conn_02x07_Odd_Even, J3 Conn_01x19, J4 Conn_01x04, J5 Conn_01x04, J6 Screw_Terminal_01x02, J7 Screw_Terminal_01x07

Commit message: kicad files for v1.2 PCB
Parts:
- added JP2, JP3: SolderJumper_2_Open, Jumper:SolderJumper-2_P1.3mm_Open_RoundedPad1.0x1.5mm, symbol Jumper:SolderJumper_2_Open
- J2: footprint Connector_PinSocket_2.54mm:PinSocket_2x07_P2.54mm_Vertical -> ct:PinSocket_2x07_P2.54_Vertical_Hybrid_SMD_THT_DBLSIDED
Connections:
- net NC: now also JP3.1 (A); no longer J3.11 (Pin_11)
- net RETCLK: now also JP2.1 (A); no longer J3.14 (Pin_14)
- net DE renamed DE/RE
- new net NC_SW: J3.11 (Pin_11), JP3.2 (B)
- new net RCLK_SW: J3.14 (Pin_14), JP2.2 (B)
Changed lines of the file:
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@@
   (title_block
     (title "ESP32 LAN8720 RS485")
-    (date "2022-09-24")
-    (rev "v1.0")
+    (date "2023-01-15")
+    (rev "v1.1")
     (company "ColossalTurtle")
   )
@@
   )
   (junction (at 180.34 72.39) (diameter 0) (color 0 0 0 0)
-  )
-  (junction (at 96.52 143.51) (diameter 0) (color 0 0 0 0)
   )
   (no_connect (at 82.55 80.01))
@@
     (stroke (width 0) (type default) (color 0 0 0 0))
   )
-  (wire (pts (xy 96.52 143.51) (xy 99.06 143.51))
-    (stroke (width 0) (type default) (color 0 0 0 0))
-  )
   (polyline (pts (xy 125.73 30.48) (xy 125.73 93.98))
     (stroke (width 0) (type default) (color 0 0 0 0))
@@
     (stroke (width 0) (type default) (color 0 0 0 0))
   )
+  (wire (pts (xy 129.54 114.3) (xy 129.54 118.11))
+    (stroke (width 0) (type default) (color 0 0 0 0))
+  )
   (wire (pts (xy 76.2 105.41) (xy 81.28 105.41))
     (stroke (width 0) (type default) (color 0 0 0 0))
@@
     (stroke (width 0) (type default) (color 0 0 0 0))
   )
+  (wire (pts (xy 138.43 104.14) (xy 138.43 106.68))
+    (stroke (width 0) (type default) (color 0 0 0 0))
+  )
+  (wire (pts (xy 138.43 114.3) (xy 138.43 118.11))
+    (stroke (width 0) (type default) (color 0 0 0 0))
+  )
   (wire (pts (xy 69.85 138.43) (xy 73.66 138.43))
     (stroke (width 0) (type default) (color 0 0 0 0))
@@
   )
   (wire (pts (xy 93.98 105.41) (xy 97.79 105.41))
+    (stroke (width 0) (type default) (color 0 0 0 0))
+  )
+  (wire (pts (xy 129.54 104.14) (xy 129.54 106.68))
     (stroke (width 0) (type default) (color 0 0 0 0))
   )
@@
     (effects (font (size 1.57 1.57)) (justify right bottom))
   )
-  (label "NC" (at 114.3 69.85 0)
-    (effects (font (size 1.27 1.27)) (justify left bottom))
-  )
   (label "NC" (at 119.38 101.6 0)
     (effects (font (size 1.27 1.27)) (justify left bottom))
@@
     (effects (font (size 1.27 1.27)) (justify left bottom))
   )
-  (label "DE" (at 99.06 140.97 0)
+  (label "DE{slash}RE" (at 99.06 140.97 0)
     (effects (font (size 1.27 1.27)) (justify left bottom))
   )
@@
     (effects (font (size 1.27 1.27)) (justify right bottom))
   )
-  (label "RE" (at 99.06 143.51 0)
+  (label "DE{slash}RE" (at 114.3 67.31 0)
     (effects (font (size 1.27 1.27)) (justify left bottom))
   )
@@
     (effects (font (size 1.27 1.27)) (justify left bottom))
   )
+  (label "NC_SW" (at 114.3 69.85 0)
+    (effects (font (size 1.27 1.27)) (justify left bottom))
+  )
   (label "TXEN" (at 76.2 118.11 180)
     (effects (font (size 1.27 1.27)) (justify right bottom))
@@
     (effects (font (size 1.27 1.27)) (justify left bottom))
   )
+  (label "RCLK_SW" (at 114.3 77.47 0)
+    (effects (font (size 1.27 1.27)) (justify left bottom))
+  )
   (label "RETCLK" (at 115.57 119.38 180)
     (effects (font (size 1.27 1.27)) (justify right bottom))
@@
     (effects (font (size 1.27 1.27)) (justify right bottom))
   )
+  (label "NC" (at 138.43 118.11 270)
+    (effects (font (size 1.27 1.27)) (justify right bottom))
+  )
   (label "3v3" (at 78.74 44.45 180)
     (effects (font (size 1.27 1.27)) (justify right bottom))
   )
-  (label "RETCLK" (at 114.3 77.47 0)
-    (effects (font (size 1.27 1.27)) (justify left bottom))
+  (label "RETCLK" (at 129.54 118.11 270)
+    (effects (font (size 1.27 1.27)) (justify right bottom))
   )
   (label "RX1" (at 78.74 67.31 180)
@@
     (effects (font (size 1.27 1.27)) (justify right bottom))
   )
+  (label "NC_SW" (at 138.43 104.14 90)
+    (effects (font (size 1.27 1.27)) (justify left bottom))
+  )
   (label "RETCLK" (at 76.2 113.03 180)
     (effects (font (size 1.27 1.27)) (justify right bottom))
@@
     (effects (font (size 1.27 1.27)) (justify right bottom))
   )
-  (label "DE" (at 114.3 67.31 0)
-    (effects (font (size 1.27 1.27)) (justify left bottom))
-  )
   (label "RO" (at 99.06 146.05 0)
     (effects (font (size 1.27 1.27)) (justify left bottom))
@@
   )
   (label "GND" (at 114.3 44.45 0)
+    (effects (font (size 1.27 1.27)) (justify left bottom))
+  )
+  (label "RCLK_SW" (at 129.54 104.14 90)
     (effects (font (size 1.27 1.27)) (justify left bottom))
   )
@@
     (property "Reference" "J2" (id 0) (at 87.63 99.06 0))
     (property "Value" "Conn_02x07_Odd_Even" (id 1) (at 87.63 101.6 0))
-    (property "Footprint" "Connector_PinSocket_2.54mm:PinSocket_2x07_P2.54mm_Vertical" (id 2) (at 86.36 113.03 0)
+    (property "Footprint" "ct:PinSocket_2x07_P2.54_Vertical_Hybrid_SMD_THT_DBLSIDED" (id 2) (at 86.36 113.03 0)
       (effects (font (size 1.27 1.27)) hide)
     )
@@
     (pin "4")
   )
+  (symbol (lib_id "Jumper:SolderJumper_2_Open") (at 138.43 110.49 90) (unit 1)
+    (in_bom yes) (on_board yes)
+    (property "Reference" "JP3" (id 0) (at 140.97 106.68 90)
+      (effects (font (size 1.27 1.27)) (justify right))
+    )
+    (property "Value" "SolderJumper_2_Open" (id 1) (at 134.62 116.84 90)
+      (effects (font (size 1.27 1.27)) (justify right) hide)
+    )
+    (property "Footprint" "Jumper:SolderJumper-2_P1.3mm_Open_RoundedPad1.0x1.5mm" (id 2) (at 138.43 110.49 0)
+      (effects (font (size 1.27 1.27)) hide)
+    )
+    (property "Datasheet" "~" (id 3) (at 138.43 110.49 0)
+      (effects (font (size 1.27 1.27)) hide)
+    )
+    (pin "1")
+    (pin "2")
+  )
   (symbol (lib_id "Connector_Generic:Conn_01x19") (at 105.41 67.31 0) (mirror y) (unit 1)
     (in_bom yes) (on_board yes) (fields_autoplaced)
@@
     (pin "1")
   )
+  (symbol (lib_id "Jumper:SolderJumper_2_Open") (at 129.54 110.49 90) (unit 1)
+    (in_bom yes) (on_board yes)
+    (property "Reference" "JP2" (id 0) (at 132.08 106.68 90)
+      (effects (font (size 1.27 1.27)) (justify right))
+    )
+    (property "Value" "SolderJumper_2_Open" (id 1) (at 125.73 116.84 90)
+      (effects (font (size 1.27 1.27)) (justify right) hide)
+    )
+    (property "Footprint" "Jumper:SolderJumper-2_P1.3mm_Open_RoundedPad1.0x1.5mm" (id 2) (at 129.54 110.49 0)
+      (effects (font (size 1.27 1.27)) hide)
+    )
+    (property "Datasheet" "~" (id 3) (at 129.54 110.49 0)
+      (effects (font (size 1.27 1.27)) hide)
+    )
+    (pin "1")
+    (pin "2")
+  )
   (symbol (lib_id "Connector:Screw_Terminal_01x07") (at 185.42 80.01 0) (unit 1)
     (in_bom yes) (on_board yes) (fields_autoplaced)
@@
     )
     (path "/137c0584-61d9-457b-ad6c-667a6a305329"
-      (reference "J2") (unit 1) (value "Conn_02x07_Odd_Even") (footprint "Connector_PinSocket_2.54mm:PinSocket_2x07_P2.54mm_Vertical")
+      (reference "J2") (unit 1) (value "Conn_02x07_Odd_Even") (footprint "ct:PinSocket_2x07_P2.54_Vertical_Hybrid_SMD_THT_DBLSIDED")
     )
     (path "/90eb17f3-bc57-4529-9492-9a5f9e436dc3"
@@
       (reference "JP1") (unit 1) (value "Jumper_3_Open") (footprint "Connector_PinHeader_2.54mm:PinHeader_1x03_P2.54mm_Vertical")
     )
+    (path "/faa59f45-f042-48ce-b2fc-fb5e4cb136f0"
+      (reference "JP2") (unit 1) (value "SolderJumper_2_Open") (footprint "Jumper:SolderJumper-2_P1.3mm_Open_RoundedPad1.0x1.5mm")
+    )
+    (path "/85e57faa-9071-44b6-8d94-b02e87621de8"
+      (reference "JP3") (unit 1) (value "SolderJumper_2_Open") (footprint "Jumper:SolderJumper-2_P1.3mm_Open_RoundedPad1.0x1.5mm")
+    )
     (path "/0d0fe49c-d812-47bf-b96f-af7b8417b02e"
